Commit message: grasp cam

File: PROBOT_Anno/probot_description/urdf/PROBOT_Anno/probot_anno_with_gripper.xacro (robot description, xacro)
@@ -206,32 +206,4 @@
     <child link="tool0" />
   </joint>
-   <joint name="camera_joint" type="fixed">
-        <origin xyz="0 0 0.05" rpy="0 ${-M_PI/2} 0"/>
-        <parent link="tool0"/>
-        <child link="camera_link"/>
-   </joint>
-   <!-- Camera -->
-   <link name="camera_link">
-       <collision>
-           <origin xyz="0 0 0" rpy="0 0 0"/>
-           <geometry>
-           <mesh filename="package://probot_description/meshes/PROBOT_Anno/sensors/camera.STL"/>
-           </geometry>
-       </collision>
-       <visual>
-           <origin xyz="0 0 0" rpy="${-M_PI} 0 ${-M_PI/2}"/>
-           <geometry>
-           <mesh filename="package://probot_description/meshes/PROBOT_Anno/sensors/camera.STL"/>
-           </geometry>
-           <material name="red"/>
-       </visual>
-       <inertial>
-        <mass value="0.00001" />
-        <origin xyz="0 0 0" />
-        <inertia ixx="1.0" ixy="0.0" ixz="0.0"
-          iyy="1.0" iyz="0.0"
-          izz="1.0" />
-       </inertial>
-   </link>
    <!-- Attach the right gripper -->
    <gripper parent="tool0" color="Green" xyz="0 0.015 0.02" rpy="0 ${-M_PI/2} ${-M_PI/2}"/>
@@ -256,46 +228,5 @@
   <xacro:transmission_block joint_name="joint_6"/>
   <xacro:transmission_block joint_name="gripper_finger_joint"/>
-  <gazebo reference="camera_link">
-    <material>Gazebo/Red</material>
-    <sensor type="camera" name="camera">
-      <update_rate>30.0</update_rate>
-      <camera name="head">
-        <horizontal_fov>1.3</horizontal_fov>
-        <!-- <horizontal_fov>0.95</horizontal_fov> -->
-        <image>
-          <width>800</width>
-          <height>800</height>
-          <format>R8G8B8</format>
-        </image>
-        <clip>
-          <near>0.02</near>
-          <far>300</far>
-        </clip>
-        <noise>
-          <type>gaussian</type>
-          <!-- Noise is sampled independently per pixel on each frame.
-               That pixel's noise value is added to each of its color
-               channels, which at that point lie in the range [0,1]. -->
-          <mean>0.0</mean>
-          <stddev>0.007</stddev>
-        </noise>
-      </camera>
-      <plugin name="camera_controller" filename="libgazebo_ros_camera.so">
-        <alwaysOn>true</alwaysOn>
-        <updateRate>0.0</updateRate>
-        <cameraName>probot_anno/camera</cameraName>
-        <imageTopicName>image_raw</imageTopicName>
-        <cameraInfoTopicName>camera_info</cameraInfoTopicName>
-        <frameName>camera_link</frameName>
-        <hackBaseline>0.07</hackBaseline>
-        <distortionK1>0.0</distortionK1>
-        <distortionK2>0.0</distortionK2>
-        <distortionK3>0.0</distortionK3>
-        <distortionT1>0.0</distortionT1>
-        <distortionT2>0.0</distortionT2>
-      </plugin>
-    </sensor>
-  </gazebo>
-  <!-- <xacro:include filename="$(find probot_description)/urdf/PROBOT_Anno/sensors/camera.urdf.xacro"/> -->
+  <xacro:include filename="$(find probot_description)/urdf/PROBOT_Anno/sensors/camera.urdf.xacro"/>
   <!-- ros_control plugin -->
   <gazebo>

File: PROBOT_Anno/probot_description/urdf/PROBOT_Anno/sensors/camera.urdf.xacro (robot description, xacro)
@@ -4,7 +4,8 @@
 -->
 <robot name="camera" xmlns:xacro="http://ros.org/wiki/xacro">
+<!-- MODIFIED -->
    <joint name="camera_joint" type="fixed">
-        <origin xyz="0.3 0 0.7" rpy="0 ${M_PI/2} 0"/>
-        <parent link="base_link"/>
+        <origin xyz="0 0.008 0.06" rpy="0 ${-M_PI/2} 0"/>
+        <parent link="tool0"/>
         <child link="camera_link"/>
    </joint>
