Commit message: 加入边缘检测与运动控制

File: PROBOT_Anno/probot_description/urdf/PROBOT_Anno/sensors/camera.urdf.xacro (robot description, xacro)
@@ -5,6 +5,6 @@
 <robot name="camera" xmlns:xacro="http://ros.org/wiki/xacro">
    <joint name="camera_joint" type="fixed">
-        <origin xyz="0.3 0 0.7" rpy="0 ${M_PI/2} 0"/>
-        <parent link="base_link"/>
+        <origin xyz="0 0.01 0.06" rpy="0 ${-M_PI/2} 0"/>
+        <parent link="tool0"/>
         <child link="camera_link"/>
    </joint>
